Commit message: functional demo, no sensor data integrated

File: training/ref/demo_manipulation/robot_config/urdf/sia20d_workspace.xacro (robot description, xacro)
@@ -8,8 +8,26 @@
 	<xacro:property name="workcell_height" value="1"/>
 	<xacro:property name="coupler_height" value="0.087"/>
+        <xacro:property name="attached_object_length" value="0.17"/>
+	<xacro:property name="attached_object_width" value="0.17"/>
+	<xacro:property name="attached_object_height" value="0.17"/>
 	<xacro:property name="arm_prefix" value=""/>
 	<!-- instantiating workcell definitions -->
 	<xacro:workcell_zone1_components/>
 	<!-- end of workcell definitions -->
+	<link name="roof1">
+		<collision>
+			<geometry>
+				<box size="0.921 2.220 0.04"/>
+			</geometry>
+		</collision>
+	</link>
+	<link name="attached_object_link">
+		<collision>
+			<geometry>
+				<box size="${attached_object_length} ${attached_object_width} ${attached_object_height}"/>
+			</geometry>
+			<material name="blue_transparent"/>
+		</collision>
+	</link>
 	<!-- instantiating sensor definitions -->
 	<xacro:sensor_definitions prefix="${arm_prefix}" parent_link="${arm_prefix}base_link"
@@ -20,8 +38,18 @@
 	<xacro:sia20d_mesh prefix="${arm_prefix}"/>
 	<!-- arm-workcell joint definitions -->
-	<joint name="wordl_to_base" type="fixed">
+	<joint name="world_to_base" type="fixed">
 		<parent link="world_frame"/>
 		<child link="${arm_prefix}base_link"/>
 		<origin xyz="0.241 0 0" rpy="0 0 0"/>
+	</joint>
+	<joint name="world_to_roof1" type="fixed">
+		<parent link="world_frame"/>
+		<child link="roof1"/>
+		<origin xyz="0.987 0 1.20" rpy="0 0 0"/>
+	</joint>
+	<joint name="tcp_to_attached_object" type="fixed">
+		<parent link="tcp_frame"/>
+		<child link="attached_object_link"/>
+		<origin xyz="0 0 ${0.5 * attached_object_height}"/>
 	</joint>
 	<!-- end of arm workcell joint definitions-->

File: training/ref/demo_manipulation/robot_config/urdf/workspace_components.xacro (robot description, xacro)
@@ -86,10 +86,12 @@
 		<xacro:workcell_element name="front_wall1" parent="world_frame"
 			 length="0.1" width="2.220" height="${workcell_height}" offset_x="1.3375" offset_y="0"/>
-		<!--xacro:workcell_element name="back_wall1" parent="world_frame"
-			 length="0.04" width="2.00" height="${workcell_height}" offset_x="0.02" offset_y="0"/-->
+		<xacro:workcell_element name="back_wall1" parent="world_frame"
+			 length="0.04" width="2.00" height="${workcell_height}" offset_x="0.02" offset_y="0"/>
 		<xacro:workcell_element name="left_wall1" parent="world_frame"
 			 length="1.221" width="0.1" height="${workcell_height}" offset_x="0.687" offset_y="1.060"/>
 		<xacro:workcell_element name="right_wall1" parent="world_frame"
 			 length="1.221" width="0.1" height="${workcell_height}" offset_x="0.687" offset_y="-1.060"/>
+		<xacro:workcell_element name="pole1" parent="world_frame"
+			length="0.09" width="0.09" height="${workcell_height}" offset_x="0.9465" offset_y="-0.845"/>
 	</xacro:macro>
 	<!-- end of workcell part1 components macro -->
