Commit message: commiting the modified files from Monday Night

File: training/ref/demo_manipulation/robot_config/urdf/sia20d_workspace.urdf (robot description, URDF)
Before this commit: robot sia20d_workspace, 29 links, 28 joints
Links:
- removed link tool0
- added link gripper_body2; collision cylinder length=0.12 radius=0.075; visual sphere radius=0.075
- link attached_object_link: geometry collision box size=0.1 0.1 0.025
- link gripper_body: geometry collision box size=0.02 0.08 0.1; collision box size=0.1 0.08 0.02
- link roof1: geometry collision box size=1.010 2.220 0.04
Joints:
- removed joint link_t-tool0
- added joint gripper_to_palm2: type fixed, parent gripper_frame, child gripper_body2, origin xyz=0 0 0.145 rpy=0 0 0
- joint coupler_to_gripper: origin xyz=0 0.087 0 rpy=-1.570 3.14 0 -> xyz=0 0 0 rpy=-1.570 3.14 0
- joint gripper_to_palm: origin xyz=0 0 0.0473 rpy=0 0 0 -> xyz=0 0 0.035 rpy=0 0 0
- joint gripper_to_tcp: origin xyz= 0 0.022 0.11 rpy=0 0 0 -> xyz= 0 0 0.19 rpy=0 0 0
- joint joint_r: limit lower=-3.1416 upper=3.1416 effort=100 velocity=3.48 -> lower=-3.00 upper=3.00 effort=100 velocity=3.48
- joint tcp_to_attached_object: origin xyz=0 0 0.085 -> xyz=0 0 0.0125

File: training/ref/demo_manipulation/robot_config/urdf/sia20d_workspace.xacro (robot description, xacro)
@@ -2,5 +2,5 @@
 <robot name="sia20d_workspace" xmlns:xacro="http://ros.org/wiki/xacro">
 	<include filename="$(find motoman_config)/cfg/sia20d_mesh_macro.xacro"/>
-	<include filename="$(find robot_config)/urdf/vacuum_gripper_macro.xacro"/>
+	<include filename="$(find robot_config)/urdf/versaball_macro.xacro"/>
 	<include filename="$(find robot_config)/urdf/workspace_components.xacro"/>
 	<include filename="$(find robot_config)/urdf/kinect_sensor_macro.xacro"/>
@@ -8,7 +8,7 @@
 	<xacro:property name="workcell_height" value="1"/>
 	<xacro:property name="coupler_height" value="0.087"/>
-        <xacro:property name="attached_object_length" value="0.17"/>
-	<xacro:property name="attached_object_width" value="0.17"/>
-	<xacro:property name="attached_object_height" value="0.17"/>
+        <xacro:property name="attached_object_length" value="0.10"/>
+	<xacro:property name="attached_object_width" value="0.10"/>
+	<xacro:property name="attached_object_height" value="0.025"/>
 	<xacro:property name="arm_prefix" value=""/>
 	<!-- instantiating workcell definitions -->
@@ -18,5 +18,5 @@
 		<collision>
 			<geometry>
-				<box size="0.921 2.220 0.04"/>
+				<box size="1.010 2.220 0.04"/>
 			</geometry>
 		</collision>
@@ -35,5 +35,5 @@
 	<!-- end of sensor definitions -->
 	<!-- instantiating arm and gripper -->
-	<xacro:vacuum_gripper_definition prefix="${arm_prefix}" gripper_adjustment="-0.01"/>
+	<xacro:versaball_definition prefix="${arm_prefix}" gripper_adjustment="-0.01"/>
 	<xacro:sia20d_mesh prefix="${arm_prefix}"/>
 	<!-- arm-workcell joint definitions -->
@@ -83,5 +83,5 @@
 		<parent link="${arm_prefix}coupler"/>
 		<child link="${arm_prefix}gripper_frame"/>
-		<origin xyz="0 ${coupler_height} 0" rpy="-1.570 3.14 0"/>
+		<origin xyz="0 0 0" rpy="-1.570 3.14 0"/>
 	</joint>
 	<!-- end of arm-gripper coupling joint definitions -->
